File: Electronics/SensorBoard/SensorBoard.kicad_pcb (KiCad board)
At the start: 2 copper layers, 28.4 x 21.3 mm, 8 parts, among them J1 Conn_01x05_Male, J2 Conn_01x05_Male, U1 TSSP58038, U2 TSSP58038, U3 TSSP58038

Commit message: unzip
Other:
- net class Default removed
